File: design/24-ch-relay-driver-kicad.kicad_pcb (KiCad board)
At the start: 2 copper layers, 75.2 x 33.8 mm, 37 parts, among them J201 USB_C_Receptacle_USB2.0, J202 5mm Screw Terminal 2-pin, J301 2.54mm 5-pin, J302 2.54mm 5-pin, J303 2.54mm 5-pin, J304 2.54mm 5-pin, J305 2.54mm 5-pin, J306 2.54mm 5-pin, U201 USBLC6-2SC6, U202 CH340N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

Commit message: Upgrade schematic to new KiCAD version.
Parts:
- removed LG101: LOGO, simtelic:simtelic-5
- removed LG102: LOGO, simtelic:simtelic-name-5
Other:
- board text removed: "simtelic.com"
