File: design/control-mod.kicad_sch (KiCad schematic)
At the start: 19 parts, among them J201 USB_C_Receptacle_USB2.0, J202 5mm Screw Terminal 2-pin, U201 USBLC6-2SC6, U202 CH340N, U203 STC15W204S

Commit message: Upgrade schematic to new KiCAD version.
Other:
- company: simtelic.com -> Dilshan R Jayakody
