File: design/output-stage.kicad_sch (KiCad schematic)
At the start: 12 parts, among them J301 2.54mm 5-pin, J302 2.54mm 5-pin, J303 2.54mm 5-pin, J304 2.54mm 5-pin, J305 2.54mm 5-pin, J306 2.54mm 5-pin, U301 TPIC6B595, U302 TPIC6B595, U303 TPIC6B595

Commit message: Upgrade schematic to new KiCAD version.
Other:
- company: simtelic.com -> Dilshan R Jayakody
